File: mBotBT.kicad_pcb (KiCad board)
At the start: 2 copper layers, 30.5 x 29.2 mm, 7 parts, among them P101 CONN_01X04, P102 CONN_01X03, U101 LM1084IT-3.3/NOPB, U102 XBEE

Commit message: Ordring to Elecrow
Parts:
- moved C101 1.27 mm to (114.3, 74.9)
Routing:
- net +5V: track 48.7 -> 49.5 mm
Changed lines of the file:
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@@
     (links 14)
     (no_connects 0)
-    (area 91.364999 63.424999 121.995001 92.785001)
+    (area 88.871667 63.424999 122.056501 92.785001)
     (thickness 1.6)
     (drawings 10)
-    (tracks 37)
+    (tracks 38)
     (zones 0)
     (modules 7)
@@
     (0 F.Cu signal)
     (31 B.Cu signal)
-    (32 B.Adhes user)
-    (33 F.Adhes user)
-    (34 B.Paste user)
-    (35 F.Paste user)
+    (32 B.Adhes user hide)
+    (33 F.Adhes user hide)
+    (34 B.Paste user hide)
+    (35 F.Paste user hide)
     (36 B.SilkS user)
     (37 F.SilkS user)
     (38 B.Mask user)
     (39 F.Mask user)
-    (40 Dwgs.User user)
-    (41 Cmts.User user)
-    (42 Eco1.User user)
-    (43 Eco2.User user)
+    (40 Dwgs.User user hide)
+    (41 Cmts.User user hide)
+    (42 Eco1.User user hide)
+    (43 Eco2.User user hide)
     (44 Edge.Cuts user)
-    (45 Margin user)
-    (46 B.CrtYd user)
-    (47 F.CrtYd user)
-    (48 B.Fab user)
-    (49 F.Fab user)
+    (45 Margin user hide)
+    (46 B.CrtYd user hide)
+    (47 F.CrtYd user hide)
+    (48 B.Fab user hide)
+    (49 F.Fab user hide)
   )
   (setup
@@
     (visible_elements 7FFFFFFF)
     (pcbplotparams
-      (layerselection 0x00030_80000001)
+      (layerselection 0x010f0_80000001)
       (usegerberextensions false)
       (excludeedgelayer true)
@@
       (outputformat 1)
       (mirror false)
-      (drillshape 1)
+      (drillshape 0)
       (scaleselection 1)
       (outputdirectory ""))
@@
   )
   (module w_smd_cap:c_0805 placed (layer F.Cu)
-    (at 113.03 74.93 270)
+    (at 114.3 74.93 270)
     (descr "SMT capacitor, 0805")
     (fp_text reference C101 (at 0 -1.905 270) (layer F.SilkS)
@@
   (gr_line (start 91.44 63.5) (end 91.44 92.71) (angle 90) (layer Edge.Cuts) (width 0.15))
   (gr_line (start 121.92 63.5) (end 91.44 63.5) (angle 90) (layer Edge.Cuts) (width 0.15))
-  (segment (start 110.72114 75.55992) (end 112.70742 75.55992) (width 0.5) (layer F.Cu) (net 1))
-  (segment (start 112.70742 75.55992) (end 113.03 75.8825) (width 0.5) (layer F.Cu) (net 1))
+  (segment (start 110.72114 75.55992) (end 113.97742 75.55992) (width 0.5) (layer F.Cu) (net 1) (status C00000))
+  (segment (start 113.97742 75.55992) (end 114.3 75.8825) (width 0.5) (layer F.Cu) (net 1) (status C00000))
+  (segment (start 114.3 75.8825) (end 114.3 77.1525) (width 0.5) (layer F.Cu) (net 1) (status 400000))
+  (segment (start 114.3 77.1525) (end 114.935 77.7875) (width 0.5) (layer F.Cu) (net 1))
   (segment (start 93.98 78.74) (end 93.98 87.63) (width 0.5) (layer F.Cu) (net 1))
-  (segment (start 114.935 77.7875) (end 113.03 75.8825) (width 0.5) (layer F.Cu) (net 1))
   (segment (start 114.935 88.9) (end 114.935 77.7875) (width 0.5) (layer F.Cu) (net 1))
   (segment (start 112.395 91.44) (end 114.935 88.9) (width 0.5) (layer F.Cu) (net 1))

Commit message: Bugfix
Parts:
- C101, C102: footprint w_smd_cap:c_0805 -> Capacitors_Tantalum_SMD:TantalC_SizeR_EIA-2012
- U101: value LM1084IT-3.3/NOPB -> TA48L033F
- moved G*** 1.15 mm to (107.4, 73.2)
Connections:
- U101 pad 1: GND -> +3V3
- U101 pad 2: +3V3 -> GND
Routing:
- net +3V3: track 15.3 -> 11.7 mm
- net GND: track 15.0 -> 17.4 mm
